File: horloge_textuelle.kicad_sch (KiCad schematic)
At the start: 1 part, among them U1 ESP32-WROOM-32D

Commit message: grosse merde que l'ia a fait parceque c'est une grosse merde de model gratuit de merde
Connections:
- net GND: now reaches U1.1 (GND), U1.15 (GND), U1.38 (GND), U1.39 (GND)
- net LED_DATA_IN: now reaches U1.12 (IO27)
Other:
- added sheet LED Matrix (led_matrix.kicad_sch)
Changed lines of the file:
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@@
 	(generator "eeschema")
 	(generator_version "10.0")
-	(paper "A4")
 	(symbol
 		(lib_id "RF_Module:ESP32-WROOM-32D")
@@
 		)
 	)
+	(sheet
+		(at 105 75)
+		(size 50 25)
+		(stroke
+			(width 0.1524)
+			(type default)
+		)
+		(fill
+			(color 0 0 0 0)
+		)
+		(property "Sheetname" "LED Matrix"
+			(at 105 73.73 0)
+			(effects
+				(font
+					(size 1.27 1.27)
+				)
+				(justify left bottom)
+			)
+		)
+		(property "Sheetfile" "led_matrix.kicad_sch"
+			(at 105 76.27 0)
+			(effects
+				(font
+					(size 1.27 1.27)
+				)
+				(justify left top)
+			)
+		)
+	)
+	(global_label "LED_DATA_IN"
+		(shape input)
+		(at 60.96 76.2 0)
+		(effects
+			(font
+				(size 1.27 1.27)
+			)
+			(justify left bottom)
+		)
+	)
+	(global_label "GND"
+		(shape input)
+		(at 45.72 93.98 0)
+		(effects
+			(font
+				(size 1.27 1.27)
+			)
+			(justify left bottom)
+		)
+	)
